Commit message: fix root joint fixed problem, now the hand can move towards the object

File: legged_lab/assets/handright9253/urdf/handright9253_simplified.urdf (robot description, URDF)
Before this commit: robot handright9253, 14 links, 13 joints
Joints:
- joint fixed: origin xyz=0.5 0.5 0.5 rpy=-1.5707963 0 0 -> xyz=0.0 0.0 0.0 rpy=-1.5707963 0 0
