Commit message: add palm center and palm dir in urdf and then usd

File: legged_lab/assets/shadow_hand_with_fingertip/shadow_hand_right.urdf (robot description, URDF)
Before this commit: robot shadow_right, 33 links, 32 joints
Links:
- added link palm_center_marker, mass 1e-06; visual sphere radius=0.01
- added link palm_dir_marker, mass 1e-06; visual box size=0.004 0.10 0.004
Joints:
- added joint center_to_dir_marker: type fixed, parent palm_center_marker, child palm_dir_marker, origin xyz=0.0 0.0 0.0 rpy=0 0 0
- added joint palm_to_center_marker: type fixed, parent palm, child palm_center_marker, origin xyz=0.0 0.0 0.0 rpy=0 0 0
