Commit message: add tendon behavior to shadow_hand urdf and converted to usd

File: legged_lab/assets/shadow_hand_with_fingertip/shadow_hand_right_for_conversion.urdf (robot description, URDF)
Before this commit: robot shadow_right, 33 links, 32 joints
Joints:
- joint FFJ1: mimic (none) -> joint=FFJ2 multiplier=1.142199 offset=0
- joint LFJ1: mimic (none) -> joint=LFJ2 multiplier=1.142199 offset=0
- joint MFJ1: mimic (none) -> joint=MFJ2 multiplier=1.142199 offset=0
- joint RFJ1: mimic (none) -> joint=RFJ2 multiplier=1.142199 offset=0
